File: PCB/SunluS1Board/SunluS1Board.kicad_sch (KiCad schematic)
At the start: 44 parts, among them J1 Conn_01x14, J2 aNTC, J3 hNTC, J4 Fan, J5 HT, J6 Power, J7 Conn_02x03_Counter_Clockwise, Q1 AO3400A, Q2 AO3400A, Q3 AO3400A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

Commit message: add current regulator to display
Parts:
- added D2: NSI45030AT1G, Diode_SMD:D_SOD-123, symbol Device:D_Current-regulator
Connections:
- net at Q3.3 (D): now also D2.1 (K); no longer J1.3 (Pin_3)
- new net: D2.2 (A), J1.3 (Pin_3)
Changed lines of the file:
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@@
 	(wire
 		(pts
-			(xy 252.73 30.48) (xy 228.6 30.48)
+			(xy 252.73 30.48) (xy 240.03 30.48)
 		)
 		(stroke
@@
 	(wire
 		(pts
+			(xy 232.41 30.48) (xy 228.6 30.48)
+		)
+		(stroke
+			(width 0)
+			(type default)
+		)
+	)
+	(wire
+		(pts
 			(xy 85.09 99.06) (xy 78.74 99.06)
 		)
@@
 					(unit 1)
 				)
+			)
+		)
+	)
+	(symbol
+		(lib_id "Device:D_Current-regulator")
+		(at 236.22 30.48 0)
+		(unit 1)
+		(exclude_from_sim no)
+		(in_bom yes)
+		(on_board yes)
+		(dnp no)
+		(fields_autoplaced yes)
+		(property "Reference" "D2"
+			(at 236.22 24.13 0)
+			(effects
+				(font
+					(size 1.27 1.27)
+				)
+			)
+		)
+		(property "Value" "NSI45030AT1G"
+			(at 236.22 26.67 0)
+			(effects
+				(font
+					(size 1.27 1.27)
+				)
+			)
+		)
+		(property "Footprint" "Diode_SMD:D_SOD-123"
+			(at 236.347 30.48 0)
+			(effects
+				(font
+					(size 1.27 1.27)
+				)
+				(hide yes)
+			)
+		)
+		(property "Datasheet" "~"
+			(at 236.22 30.48 0)
+			(effects
+				(font
+					(size 1.27 1.27)
+				)
+				(hide yes)
+			)
+		)
+		(property "Description" "Constant-current diode / current limiting diode / current regulator diode, IEC60747-3:2013"
+			(at 236.22 30.48 0)
+			(effects
+				(font
+					(size 1.27 1.27)
+				)
+				(hide yes)
+			)
+		)
+		(pin "2"
+		)
+		(pin "1"
+		)
+		(instances
+			(project ""
+				(path "/2863b0a4-ce41-4b5d-85c6-a6fe5f63d9f6"
+					(reference "D2")
+					(unit 1)
+				)

Commit message: add resistor fallback
Parts:
- added R13: 22, symbol Device:R
Connections:
- net at D2.1 (K), Q3.3 (D): now also R13.2
- net at D2.2 (A), J1.3 (Pin_3): now also R13.1
Changed lines of the file:
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@@
+	)
+	(junction
+		(at 228.6 30.48)
+		(diameter 0)
+		(color 0 0 0 0)
 	)
 	(junction
@@
 		(color 0 0 0 0)
 	)
+	(junction
+		(at 243.84 30.48)
+		(diameter 0)
+		(color 0 0 0 0)
+	)
 	(no_connect
 		(at 252.73 25.4)
@@
 	(wire
 		(pts
+			(xy 232.41 20.32) (xy 228.6 20.32)
+		)
+		(stroke
+			(width 0)
+			(type default)
+		)
+	)
+	(wire
+		(pts
+			(xy 228.6 20.32) (xy 228.6 30.48)
+		)
+		(stroke
+			(width 0)
+			(type default)
+		)
+	)
+	(wire
+		(pts
 			(xy 80.01 168.91) (xy 80.01 172.72)
 		)
@@
 	(wire
 		(pts
+			(xy 243.84 30.48) (xy 240.03 30.48)
+		)
+		(stroke
+			(width 0)
+			(type default)
+		)
+	)
+	(wire
+		(pts
 			(xy 228.6 66.04) (xy 228.6 63.5)
 		)
@@
 	(wire
 		(pts
-			(xy 252.73 30.48) (xy 240.03 30.48)
+			(xy 252.73 30.48) (xy 243.84 30.48)
 		)
 		(stroke
@@
 	(wire
 		(pts
+			(xy 243.84 20.32) (xy 243.84 30.48)
+		)
+		(stroke
+			(width 0)
+			(type default)
+		)
+	)
+	(wire
+		(pts
 			(xy 171.45 40.64) (xy 171.45 46.99)
 		)
@@
 		(pts
 			(xy 102.87 168.91) (xy 102.87 172.72)
+		)
+		(stroke
+			(width 0)
+			(type default)
+		)
+	)
+	(wire
+		(pts
+			(xy 240.03 20.32) (xy 243.84 20.32)
 		)
 		(stroke
@@
 					(unit 1)
 				)
+			)
+		)
+	)
+	(symbol
+		(lib_id "Device:R")
+		(at 236.22 20.32 270)
+		(unit 1)
+		(exclude_from_sim no)
+		(in_bom yes)
+		(on_board yes)
+		(dnp yes)
+		(fields_autoplaced yes)
+		(property "Reference" "R13"
+			(at 236.22 13.97 90)
+			(effects
+				(font
+					(size 1.27 1.27)
+				)
+			)
+		)
+		(property "Value" "22"
+			(at 236.22 16.51 90)
+			(effects
+				(font
+					(size 1.27 1.27)
+				)
+			)
+		)
+		(property "Footprint" ""
+			(at 236.22 18.542 90)
+			(effects
+				(font
+					(size 1.27 1.27)
+				)
+				(hide yes)
+			)
+		)
+		(property "Datasheet" "~"
+			(at 236.22 20.32 0)
+			(effects
+				(font
+					(size 1.27 1.27)
+				)
+				(hide yes)
+			)
+		)
+		(property "Description" "Resistor"
+			(at 236.22 20.32 0)
+			(effects
+				(font
+					(size 1.27 1.27)
+				)
+				(hide yes)
+			)
+		)
+		(pin "2"
+		)
+		(pin "1"
+		)
+		(instances
+			(project "SunluS1Board"
+				(path "/2863b0a4-ce41-4b5d-85c6-a6fe5f63d9f6"
+					(reference "R13")
+					(unit 1)
+				)

Commit message: finish schematic fr
Parts:
- removed TH1: 100k, symbol Device:Thermistor_NTC
- removed TH2: Thermistor_NTC, symbol Device:Thermistor_NTC
- added D3: 1N4007W, Diode_SMD:Nexperia_CFP3_SOD-123W, symbol Diode:1N4007
- C1, C11, C12, C14, C2, C3, C5, C7, C9: footprint (none) -> Capacitor_SMD:C_0603_1608Metric
- C10, C6: value 10uF -> 1uF; footprint (none) -> Capacitor_SMD:C_0805_2012Metric
- C13, C4, C8: value 10uF -> 1uF; footprint (none) -> Capacitor_SMD:C_0603_1608Metric
- D1: footprint (none) -> LED_SMD:LED_0603_1608Metric
- J2, J3: footprint (none) -> Connector_Molex:Molex_PicoBlade_53048-0210_1x02_P1.25mm_Horizontal
- R1, R10, R11, R12, R13, R2, R3, R4, R5, R6, R7, R8, R9: footprint (none) -> Resistor_SMD:R_0603_1608Metric
Connections:
- net +24V: now also D3.2 (A); no longer U2.1 (VI)
- new net: D3.1 (K), U2.1 (VI)
Other:
- moved on the sheet: F1
