File: PCB/SunluS1Board/SunluS1Board.kicad_sch (KiCad schematic)
At the start: 56 parts, among them J1 Conn_01x14, J2 aNTC, J3 hNTC, J4 Fan, J5 HT, J6 Power, J7 Conn_02x03_Odd_Even, Q1 SIA440DJ-T1-GE3, Q2 AO3400A, Q3 AO3400A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

Commit message: footprints
Parts:
- removed D4: D_Schottky, symbol Device:D_Schottky
- added D3: B360, Diode_SMD:D_SMC, symbol Diode:B360
- C16: footprint (none) -> Capacitor_THT:CP_Radial_D6.3mm_P2.50mm
- C17, C21, C22: footprint (none) -> Capacitor_SMD:C_0603_1608Metric
- C18, C19: footprint (none) -> Capacitor_SMD:C_0805_2012Metric
- C20: footprint (none) -> Capacitor_SMD:C_1210_3225Metric
- C5: value 1uF -> 0.1uF; footprint (none) -> Capacitor_SMD:C_0603_1608Metric
- R14, R15, R16, R17, R18, R19: footprint (none) -> Resistor_SMD:R_0603_1608Metric
Connections:
- net GND: now also D3.2 (A)
- net at C17.1, L1.1, U3.10 (PH): now also D3.1 (K)
Changed lines of the file:
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@@
 	)
 	(junction
-		(at 184.15 101.6)
+		(at 248.92 107.95)
 		(diameter 0)
 		(color 0 0 0 0)
 	)
 	(junction
-		(at 234.95 100.33)
+		(at 184.15 101.6)
 		(diameter 0)
 		(color 0 0 0 0)
 	)
 	(junction
-		(at 33.02 162.56)
+		(at 234.95 100.33)
 		(diameter 0)
 		(color 0 0 0 0)
 	)
 	(junction
-		(at 248.92 107.95)
+		(at 33.02 162.56)
 		(diameter 0)
 		(color 0 0 0 0)
@@
 	)
 	(junction
-		(at 248.92 100.33)
+		(at 102.87 152.4)
 		(diameter 0)
 		(color 0 0 0 0)
 	)
 	(junction
-		(at 102.87 152.4)
+		(at 90.17 63.5)
 		(diameter 0)
 		(color 0 0 0 0)
 	)
 	(junction
-		(at 90.17 63.5)
+		(at 248.92 100.33)
 		(diameter 0)
 		(color 0 0 0 0)
@@
 	(wire
 		(pts
+			(xy 248.92 107.95) (xy 265.43 107.95)
+		)
+		(stroke
+			(width 0)
+			(type default)
+		)
+	)
+	(wire
+		(pts
 			(xy 232.41 107.95) (xy 232.41 106.68)
 		)
@@
 	(wire
 		(pts
-			(xy 234.95 107.95) (xy 248.92 107.95)
-		)
-		(stroke
-			(width 0)
-			(type default)
-		)
-	)
-	(wire
-		(pts
 			(xy 193.04 143.51) (xy 193.04 139.7)
 		)
@@
 	(wire
 		(pts
-			(xy 248.92 100.33) (xy 234.95 100.33)
+			(xy 248.92 100.33) (xy 250.19 100.33)
 		)
 		(stroke
@@
 	(wire
 		(pts
-			(xy 250.19 100.33) (xy 248.92 100.33)
+			(xy 234.95 100.33) (xy 248.92 100.33)
 		)
 		(stroke
@@
 	(wire
 		(pts
-			(xy 248.92 107.95) (xy 265.43 107.95)
+			(xy 234.95 107.95) (xy 248.92 107.95)
 		)
 		(stroke
@@
 			)
 		)
-		(property "Footprint" ""
+		(property "Footprint" "Capacitor_SMD:C_1210_3225Metric"
 			(at 172.4152 109.22 0)
 			(effects
@@
 			)
 		)
-		(property "Value" "1uF"
+		(property "Value" "0.1uF"
 			(at 163.068 106.68 0)
 			(effects
@@
 			)
 		)
-		(property "Footprint" ""
+		(property "Footprint" "Capacitor_SMD:C_0603_1608Metric"
 			(at 160.9852 109.22 0)
 			(effects
@@
 			)
 		)
-		(property "Footprint" ""
+		(property "Footprint" "Capacitor_SMD:C_0603_1608Metric"
 			(at 194.0052 139.7 0)
 			(effects
@@
 			)
 		)
-		(property "Footprint" ""
+		(property "Footprint" "Resistor_SMD:R_0603_1608Metric"
 			(at 182.372 105.41 90)
 			(effects
@@
 	)
 	(symbol
+		(lib_id "Diode:B360")
+		(at 248.92 104.14 270)
+		(unit 1)
+		(exclude_from_sim no)
+		(in_bom yes)
+		(on_board yes)
+		(dnp no)
+		(fields_autoplaced yes)
+		(property "Reference" "D3"
+			(at 251.46 102.5524 90)
+			(effects
+				(font
+					(size 1.27 1.27)
+				)
+				(justify left)
+			)
+		)
+		(property "Value" "B360"
+			(at 251.46 105.0924 90)
+			(effects
+				(font
+					(size 1.27 1.27)
+				)
+				(justify left)
+			)
+		)
+		(property "Footprint" "Diode_SMD:D_SMC"
+			(at 244.475 104.14 0)
+			(effects
+				(font
+					(size 1.27 1.27)
+				)
+				(hide yes)
+			)
+		)
+		(property "Datasheet" "http://www.jameco.com/Jameco/Products/ProdDS/1538777.pdf"
+			(at 248.92 104.14 0)
+			(effects
+				(font
+					(size 1.27 1.27)
+				)
+				(hide yes)
+			)
+		)
+		(property "Description" "60V 3A Schottky Barrier Rectifier Diode, SMC"
+			(at 248.92 104.14 0)
+			(effects
+				(font
+					(size 1.27 1.27)
+				)
+				(hide yes)
+			)
+		)
+		(pin "2"
+		)
+		(pin "1"
+		)
+		(instances
+			(project ""
+				(path "/2863b0a4-ce41-4b5d-85c6-a6fe5f63d9f6"
+					(reference "D3")
+					(unit 1)
+				)
+			)
+		)
+	)
+	(symbol
 		(lib_id "Device:C")
 		(at 59.69 162.56 90)
@@
 			)
 		)
-		(property "Footprint" ""
+		(property "Footprint" "Resistor_SMD:R_0603_1608Metric"
 			(at 182.372 113.03 90)
 			(effects
@@
 			)
 		)
-		(property "Footprint" ""
+		(property "Footprint" "Capacitor_SMD:C_0603_1608Metric"
 			(at 235.9152 107.95 0)
 			(effects
@@
 			)
 		)
-		(property "Footprint" ""
+		(property "Footprint" "Capacitor_SMD:C_0805_2012Metric"
 			(at 279.0952 107.95 0)
 			(effects
@@
 			)
 		)
-		(property "Footprint" ""
+		(property "Footprint" "Resistor_SMD:R_0603_1608Metric"
 			(at 239.522 119.38 90)
 			(effects
@@
 			)
 		)
-		(property "Footprint" ""
+		(property "Footprint" "Capacitor_SMD:C_0805_2012Metric"
 			(at 266.3952 107.95 0)
 			(effects
@@
 			)
 		)
-		(property "Footprint" ""
+		(property "Footprint" "Capacitor_SMD:C_0603_1608Metric"
 			(at 219.4052 143.51 0)
 			(effects
@@
 			)
 		)
-		(property "Footprint" ""
+		(property "Footprint" "Resistor_SMD:R_0603_1608Metric"
 			(at 246.38 112.522 90)
 			(effects
@@
 			)
 		)
-		(property "Footprint" ""
+		(property "Footprint" "Resistor_SMD:R_0603_1608Metric"
 			(at 216.662 132.08 90)
 			(effects
@@
 	)
 	(symbol
-		(lib_id "Device:D_Schottky")
-		(at 248.92 104.14 270)
-		(unit 1)
-		(exclude_from_sim no)
-		(in_bom yes)
-		(on_board yes)
-		(dnp no)
-		(fields_autoplaced yes)
-		(property "Reference" "D4"
-			(at 251.46 102.5524 90)
-			(effects
-				(font
-					(size 1.27 1.27)
-				)
-				(justify left)
-			)
-		)
-		(property "Value" "D_Schottky"
-			(at 251.46 105.0924 90)
-			(effects
-				(font
-					(size 1.27 1.27)
-				)
-				(justify left)
-			)
-		)
-		(property "Footprint" ""
-			(at 248.92 104.14 0)
-			(effects
-				(font
-					(size 1.27 1.27)
-				)
-				(hide yes)
-			)
-		)
-		(property "Datasheet" "~"
-			(at 248.92 104.14 0)
-			(effects
-				(font
-					(size 1.27 1.27)
-				)
-				(hide yes)
-			)
-		)
-		(property "Description" "Schottky diode"
-			(at 248.92 104.14 0)
-			(effects
-				(font
-					(size 1.27 1.27)
-				)
-				(hide yes)
-			)
-		)
-		(pin "1"
-		)
-		(pin "2"
-		)
-		(instances
-			(project ""
-				(path "/2863b0a4-ce41-4b5d-85c6-a6fe5f63d9f6"
-					(reference "D4")
-					(unit 1)
-				)
-			)
-		)
-	)
-	(symbol
 		(lib_id "Connector_Generic:Conn_01x02")
 		(at 115.57 177.8 0)
@@
 			)
 		)
-		(property "Footprint" ""
+		(property "Footprint" "Capacitor_THT:CP_Radial_D6.3mm_P2.50mm"
 			(at 123.19 166.6748 0)
 			(effects
@@
 			)
 		)
-		(property "Footprint" ""
+		(property "Footprint" "Resistor_SMD:R_0603_1608Metric"
 			(at 203.962 135.89 90)
 			(effects

Commit message: fixes
Parts:
- D3: footprint Diode_SMD:D_SMC -> Diode_SMD:D_SMB
- L1: footprint (none) -> Inductor_SMD:L_APV_ANR4020
Connections:
- net GND: no longer C17.2, U3.1 (BOOT)
- new net: C17.2, U3.1 (BOOT)
Changed lines of the file:
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@@
 	)
 	(junction
-		(at 234.95 107.95)
-		(diameter 0)
-		(color 0 0 0 0)
-	)
-	(junction
 		(at 241.3 114.3)
 		(diameter 0)
@@
 	)
 	(junction
-		(at 248.92 107.95)
-		(diameter 0)
-		(color 0 0 0 0)
-	)
-	(junction
 		(at 184.15 101.6)
 		(diameter 0)
@@
 	(wire
 		(pts
-			(xy 234.95 107.95) (xy 248.92 107.95)
-		)
-		(stroke
-			(width 0)
-			(type default)
-		)
-	)
-	(wire
-		(pts
 			(xy 110.49 167.64) (xy 110.49 168.91)
 		)
@@
 			)
 		)
-		(property "Footprint" "Diode_SMD:D_SMC"
+		(property "Footprint" "Diode_SMD:D_SMB"
 			(at 244.475 104.14 0)
 			(effects
@@
 			)
 		)
-		(property "Footprint" ""
+		(property "Footprint" "Inductor_SMD:L_APV_ANR4020"
 			(at 254 100.33 0)
 			(effects

Commit message: finish V2
Parts:
- removed C16: 100uF, Capacitor_THT:CP_Radial_D6.3mm_P2.50mm, symbol Device:C_Polarized
- added C6: 100uF, easyeda2kicad:CAP-SMD_BD6.3-L6.6-W6.6-FD, symbol Device:C_Polarized
Connections:
- net +24V: now also C6.1
- net GND: now also C6.2
Changed lines of the file:
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@@
+	)
+	(symbol
+		(lib_id "Device:C_Polarized")
+		(at 119.38 167.64 90)
+		(unit 1)
+		(exclude_from_sim no)
+		(in_bom yes)
+		(on_board yes)
+		(dnp no)
+		(property "Reference" "C6"
+			(at 119.38 160.782 90)
+			(effects
+				(font
+					(size 1.27 1.27)
+				)
+			)
+		)
+		(property "Value" "100uF"
+			(at 119.38 163.322 90)
+			(effects
+				(font
+					(size 1.27 1.27)
+				)
+			)
+		)
+		(property "Footprint" "easyeda2kicad:CAP-SMD_BD6.3-L6.6-W6.6-FD"
+			(at 123.19 166.6748 0)
+			(effects
+				(font
+					(size 1.27 1.27)
+				)
+				(hide yes)
+			)
+		)
+		(property "Datasheet" "~"
+			(at 119.38 167.64 0)
+			(effects
+				(font
+					(size 1.27 1.27)
+				)
+				(hide yes)
+			)
+		)
+		(property "Description" "Polarized capacitor"
+			(at 119.38 167.64 0)
+			(effects
+				(font
+					(size 1.27 1.27)
+				)
+				(hide yes)
+			)
+		)
+		(pin "1"
+		)
+		(pin "2"
+		)
+		(instances
+			(project "SunluS1Board"
+				(path "/2863b0a4-ce41-4b5d-85c6-a6fe5f63d9f6"
+					(reference "C6")
+					(unit 1)
+				)
+			)
+		)
 	)
 	(symbol
@@
 					(unit 1)
 				)
-			)
-		)
-	)
-	(symbol
-		(lib_id "Device:C_Polarized")
-		(at 119.38 167.64 90)
-		(unit 1)
-		(exclude_from_sim no)
-		(in_bom yes)
-		(on_board yes)
-		(dnp no)
-		(property "Reference" "C16"
-			(at 119.38 160.782 90)
-			(effects
-				(font
-					(size 1.27 1.27)
-				)
-			)
-		)
-		(property "Value" "100uF"
-			(at 119.38 163.322 90)
-			(effects
-				(font
-					(size 1.27 1.27)
-				)
-			)
-		)
-		(property "Footprint" "Capacitor_THT:CP_Radial_D6.3mm_P2.50mm"
-			(at 123.19 166.6748 0)
-			(effects
-				(font
-					(size 1.27 1.27)
-				)
-				(hide yes)
-			)
-		)
-		(property "Datasheet" "~"
-			(at 119.38 167.64 0)
-			(effects
-				(font
-					(size 1.27 1.27)
-				)
-				(hide yes)
-			)
-		)
-		(property "Description" "Polarized capacitor"
-			(at 119.38 167.64 0)
-			(effects
-				(font
-					(size 1.27 1.27)
-				)
-				(hide yes)
-			)
-		)
-		(pin "1"
-		)
-		(pin "2"
-		)
-		(instances
-			(project ""
-				(path "/2863b0a4-ce41-4b5d-85c6-a6fe5f63d9f6"
-					(reference "C16")
-					(unit 1)
-				)

Commit message: fix
Parts:
- C17, C5: value 0.1uF -> 100nF
Changed lines of the file:
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@@
 			)
 		)
-		(property "Value" "0.1uF"
+		(property "Value" "100nF"
 			(at 163.068 106.68 0)
 			(effects
@@
 			)
 		)
-		(property "Value" "0.1uF"
+		(property "Value" "100nF"
 			(at 238.76 105.4099 0)
 			(effects

Commit message: finish pcb and BOM
Parts:
- C6: value 100uF -> 47uF
Changed lines of the file:
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@@
 			)
 		)
-		(property "Value" "100uF"
+		(property "Value" "47uF"
 			(at 119.38 163.322 90)
 			(effects

Commit message: Fixes for V2
Parts:
- added D4, D5: SS34, Diode_SMD:D_SMA, symbol Diode:SS34
- D2: now not fitted
- J4, J5, J6: footprint Connector_JST:JST_XH_S2B-XH-A-1_1x02_P2.50mm_Horizontal -> easyeda2kicad:CONN-TH_2P-P2.54_AXH-2AW-11
- R13: now fitted
Connections:
- net +24V: now also D4.1 (K), D5.1 (K)
- net fCon: now also D4.2 (A)
- net hCon: now also D5.2 (A)
Other:
- moved on the sheet: C10, C11, C12, C6, C9, F1, J2, J3, J5, J6, R1, R11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
