File: PCB/SunluS1Board/_autosave-SunluS1Board.kicad_sch (KiCad schematic)
At the start: 45 parts, among them J1 Conn_01x14, J2 aNTC, J3 hNTC, J4 Fan, J5 HT, J6 Power, J7 Conn_02x03_Odd_Even, Q2 AO3400A, Q3 AO3400A, Q4 SIA440DJ-T1-GE3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

Commit message: continue PCB
Parts:
- removed Q4: SIA440DJ-T1-GE3, easyeda2kicad:SC-70-6L_L2.0-W2.0-P0.65-BL, symbol easyeda2kicad:SIA440DJ-T1-GE3
- added Q1: SIA440DJ-T1-GE3, easyeda2kicad:SC-70-6L_L2.0-W2.0-P0.65-BL, symbol easyeda2kicad:SIA440DJ-T1-GE3
Connections:
- net GND: now also Q1.4 (S), Q1.7 (S)
- net hCon: now also Q1.1 (D), Q1.2 (D), Q1.5 (D), Q1.6 (D), Q1.8 (D)
- net at R2.1, R3.2: now also Q1.3 (G)
Changed lines of the file:
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@@
 	)
 	(junction
-		(at 26.67 102.87)
-		(diameter 0)
-		(color 0 0 0 0)
-	)
-	(junction
 		(at 171.45 40.64)
 		(diameter 0)
@@
 	)
 	(junction
-		(at 41.91 102.87)
-		(diameter 0)
-		(color 0 0 0 0)
-	)
-	(junction
 		(at 236.22 109.22)
 		(diameter 0)
@@
 	)
 	(junction
-		(at 41.91 107.95)
-		(diameter 0)
-		(color 0 0 0 0)
-	)
-	(junction
 		(at 149.86 147.32)
 		(diameter 0)
@@
 	)
 	(junction
+		(at 26.67 102.87)
+		(diameter 0)
+		(color 0 0 0 0)
+	)
+	(junction
 		(at 130.81 83.82)
 		(diameter 0)
@@
 	)
 	(junction
-		(at 171.45 35.56)
+		(at 41.91 102.87)
 		(diameter 0)
 		(color 0 0 0 0)
 	)
 	(junction
-		(at 34.29 113.03)
+		(at 41.91 107.95)
+		(diameter 0)
+		(color 0 0 0 0)
+	)
+	(junction
+		(at 171.45 35.56)
 		(diameter 0)
 		(color 0 0 0 0)
@@
 		(color 0 0 0 0)
 	)
+	(junction
+		(at 34.29 113.03)
+		(diameter 0)
+		(color 0 0 0 0)
+	)
 	(no_connect
 		(at 252.73 25.4)
@@
 	(wire
 		(pts
+			(xy 41.91 102.87) (xy 41.91 105.41)
+		)
+		(stroke
+			(width 0)
+			(type default)
+		)
+	)
+	(wire
+		(pts
 			(xy 266.7 101.6) (xy 273.05 101.6)
 		)
@@
 	(wire
 		(pts
-			(xy 26.67 97.79) (xy 26.67 102.87)
-		)
-		(stroke
-			(width 0)
-			(type default)
-		)
-	)
-	(wire
-		(pts
 			(xy 34.29 119.38) (xy 34.29 116.84)
 		)
@@
 	(wire
 		(pts
-			(xy 41.91 102.87) (xy 41.91 97.79)
+			(xy 41.91 97.79) (xy 41.91 102.87)
 		)
 		(stroke
@@
 	(wire
 		(pts
-			(xy 41.91 105.41) (xy 41.91 102.87)
-		)
-		(stroke
-			(width 0)
-			(type default)
-		)
-	)
-	(wire
-		(pts
 			(xy 157.48 162.56) (xy 157.48 163.83)
 		)
@@
 	(wire
 		(pts
+			(xy 26.67 97.79) (xy 26.67 102.87)
+		)
+		(stroke
+			(width 0)
+			(type default)
+		)
+	)
+	(wire
+		(pts
 			(xy 274.32 33.02) (xy 269.24 33.02)
 		)
@@
 	)
 	(symbol
+		(lib_id "easyeda2kicad:SIA440DJ-T1-GE3")
+		(at 34.29 105.41 0)
+		(mirror y)
+		(unit 1)
+		(exclude_from_sim no)
+		(in_bom yes)
+		(on_board yes)
+		(dnp no)
+		(property "Reference" "Q1"
+			(at 32.1467 95.25 0)
+			(effects
+				(font
+					(size 1.27 1.27)
+				)
+				(justify left)
+			)
+		)
+		(property "Value" "SIA440DJ-T1-GE3"
+			(at 53.594 94.742 0)
+			(effects
+				(font
+					(size 1.27 1.27)
+				)
+				(justify left)
+			)
+		)
+		(property "Footprint" "easyeda2kicad:SC-70-6L_L2.0-W2.0-P0.65-BL"
+			(at 34.29 120.65 0)
+			(effects
+				(font
+					(size 1.27 1.27)
+				)
+				(hide yes)
+			)
+		)
+		(property "Datasheet" ""
+			(at 34.29 105.41 0)
+			(effects
+				(font
+					(size 1.27 1.27)
+				)
+				(hide yes)
+			)
+		)
+		(property "Description" ""
+			(at 34.29 105.41 0)
+			(effects
+				(font
+					(size 1.27 1.27)
+				)
+				(hide yes)
+			)
+		)
+		(property "LCSC Part" "C727349"
+			(at 34.29 123.19 0)
+			(effects
+				(font
+					(size 1.27 1.27)
+				)
+				(hide yes)
+			)
+		)
+		(pin "4"
+		)
+		(pin "6"
+		)
+		(pin "5"
+		)
+		(pin "7"
+		)
+		(pin "1"
+		)
+		(pin "8"
+		)
+		(pin "3"
+		)
+		(pin "2"
+		)
+		(instances
+			(project "SunluS1Board"
+				(path "/2863b0a4-ce41-4b5d-85c6-a6fe5f63d9f6"
+					(reference "Q1")
+					(unit 1)
+				)
+			)
+		)
+	)
+	(symbol
 		(lib_id "Diode:1N4007")
 		(at 237.49 91.44 180)
@@
 					(unit 1)
 				)
-			)
-		)
-	)
-	(symbol
-		(lib_id "easyeda2kicad:SIA440DJ-T1-GE3")
-		(at 34.29 105.41 0)
-		(mirror y)
-		(unit 1)
-		(exclude_from_sim no)
-		(in_bom yes)
-		(on_board yes)
-		(dnp no)
-		(property "Reference" "Q4"
-			(at 32.1467 95.25 0)
-			(effects
-				(font
-					(size 1.27 1.27)
-				)
-				(justify left)
-			)
-		)
-		(property "Value" "SIA440DJ-T1-GE3"
-			(at 53.594 94.742 0)
-			(effects
-				(font
-					(size 1.27 1.27)
-				)
-				(justify left)
-			)
-		)
-		(property "Footprint" "easyeda2kicad:SC-70-6L_L2.0-W2.0-P0.65-BL"
-			(at 34.29 120.65 0)
-			(effects
-				(font
-					(size 1.27 1.27)
-				)
-				(hide yes)
-			)
-		)
-		(property "Datasheet" ""
-			(at 34.29 105.41 0)
-			(effects
-				(font
-					(size 1.27 1.27)
-				)
-				(hide yes)
-			)
-		)
-		(property "Description" ""
-			(at 34.29 105.41 0)
-			(effects
-				(font
-					(size 1.27 1.27)
-				)
-				(hide yes)
-			)
-		)
-		(property "LCSC Part" "C727349"
-			(at 34.29 123.19 0)
-			(effects
-				(font
-					(size 1.27 1.27)
-				)
-				(hide yes)
-			)
-		)
-		(pin "4"
-		)
-		(pin "6"
-		)
-		(pin "5"
-		)
-		(pin "7"
-		)
-		(pin "1"
-		)
-		(pin "8"
-		)
-		(pin "3"
-		)
-		(pin "2"
-		)
-		(instances
-			(project ""
-				(path "/2863b0a4-ce41-4b5d-85c6-a6fe5f63d9f6"
-					(reference "Q4")
-					(unit 1)
-				)
