File: PCB/SunluS1Board/_autosave-SunluS1Board.kicad_sch (KiCad schematic)
At the start: 45 parts, among them J1 Conn_01x14, J7 Conn_02x03_Odd_Even, Q1 SIA440DJ-T1-GE3, Q2 AO3400A, Q3 AO3400A, SW1 CS1213AGF260, SW2 CS1213AGF260, U1 STM32C011F4Px, U2 AP7381-33SA-7

Commit message: continue routing
Parts:
- renumbered HT to HT1, Vin to Vin1, aNTC to aNTC1, hNTC to hNTC1
Changed lines of the file:
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@@
 		(dnp no)
 		(fields_autoplaced yes)
-		(property "Reference" "HT"
+		(property "Reference" "HT1"
 			(at 151.13 172.7199 0)
 			(effects
@@
 			(project "SunluS1Board"
 				(path "/2863b0a4-ce41-4b5d-85c6-a6fe5f63d9f6"
-					(reference "HT")
+					(reference "HT1")
 					(unit 1)
 				)
@@
 		(dnp no)
 		(fields_autoplaced yes)
-		(property "Reference" "hNTC"
+		(property "Reference" "hNTC1"
 			(at 110.49 172.7199 0)
 			(effects
@@
 			(project "SunluS1Board"
 				(path "/2863b0a4-ce41-4b5d-85c6-a6fe5f63d9f6"
-					(reference "hNTC")
+					(reference "hNTC1")
 					(unit 1)
 				)
@@
 		(dnp no)
 		(fields_autoplaced yes)
-		(property "Reference" "aNTC"
+		(property "Reference" "aNTC1"
 			(at 87.63 172.7199 0)
 			(effects
@@
 			(project ""
 				(path "/2863b0a4-ce41-4b5d-85c6-a6fe5f63d9f6"
-					(reference "aNTC")
+					(reference "aNTC1")
 					(unit 1)
 				)
@@
 		(dnp no)
 		(fields_autoplaced yes)
-		(property "Reference" "Vin"
+		(property "Reference" "Vin1"
 			(at 165.1 172.7199 0)
 			(effects
@@
 			(project "SunluS1Board"
 				(path "/2863b0a4-ce41-4b5d-85c6-a6fe5f63d9f6"
-					(reference "Vin")
+					(reference "Vin1")
 					(unit 1)
 				)
