File: PCB/SunluS1Board/_autosave-SunluS1Board.kicad_sch (KiCad schematic)
At the start: 56 parts, among them J1 Conn_01x14, J2 aNTC, J3 hNTC, J4 Fan, J5 HT, J6 Power, J7 Conn_02x03_Odd_Even, Q1 SIA440DJ-T1-GE3, Q2 AO3400A, Q3 AO3400A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

Commit message: fixes
Parts:
- removed D4: D_Schottky, symbol Device:D_Schottky
- added D3: B360, Diode_SMD:D_SMC, symbol Diode:B360
Connections:
- net GND: now also D3.2 (A)
- net at C17.1, L1.1, U3.10 (PH): now also D3.1 (K)
Changed lines of the file:
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@@
 	)
 	(junction
-		(at 184.15 101.6)
+		(at 248.92 107.95)
 		(diameter 0)
 		(color 0 0 0 0)
 	)
 	(junction
-		(at 234.95 100.33)
+		(at 184.15 101.6)
 		(diameter 0)
 		(color 0 0 0 0)
 	)
 	(junction
-		(at 33.02 162.56)
+		(at 234.95 100.33)
 		(diameter 0)
 		(color 0 0 0 0)
 	)
 	(junction
-		(at 248.92 107.95)
+		(at 33.02 162.56)
 		(diameter 0)
 		(color 0 0 0 0)
@@
 	)
 	(junction
-		(at 248.92 100.33)
+		(at 102.87 152.4)
 		(diameter 0)
 		(color 0 0 0 0)
 	)
 	(junction
-		(at 102.87 152.4)
+		(at 90.17 63.5)
 		(diameter 0)
 		(color 0 0 0 0)
 	)
 	(junction
-		(at 90.17 63.5)
+		(at 248.92 100.33)
 		(diameter 0)
 		(color 0 0 0 0)
@@
 	(wire
 		(pts
+			(xy 248.92 107.95) (xy 265.43 107.95)
+		)
+		(stroke
+			(width 0)
+			(type default)
+		)
+	)
+	(wire
+		(pts
 			(xy 232.41 107.95) (xy 232.41 106.68)
 		)
@@
 	(wire
 		(pts
-			(xy 234.95 107.95) (xy 248.92 107.95)
-		)
-		(stroke
-			(width 0)
-			(type default)
-		)
-	)
-	(wire
-		(pts
 			(xy 193.04 143.51) (xy 193.04 139.7)
 		)
@@
 	(wire
 		(pts
-			(xy 248.92 100.33) (xy 234.95 100.33)
+			(xy 248.92 100.33) (xy 250.19 100.33)
 		)
 		(stroke
@@
 	(wire
 		(pts
-			(xy 250.19 100.33) (xy 248.92 100.33)
+			(xy 234.95 100.33) (xy 248.92 100.33)
 		)
 		(stroke
@@
 	(wire
 		(pts
-			(xy 248.92 107.95) (xy 265.43 107.95)
+			(xy 234.95 107.95) (xy 248.92 107.95)
 		)
 		(stroke
@@
 	)
 	(symbol
+		(lib_id "Diode:B360")
+		(at 248.92 104.14 270)
+		(unit 1)
+		(exclude_from_sim no)
+		(in_bom yes)
+		(on_board yes)
+		(dnp no)
+		(fields_autoplaced yes)
+		(property "Reference" "D3"
+			(at 251.46 102.5524 90)
+			(effects
+				(font
+					(size 1.27 1.27)
+				)
+				(justify left)
+			)
+		)
+		(property "Value" "B360"
+			(at 251.46 105.0924 90)
+			(effects
+				(font
+					(size 1.27 1.27)
+				)
+				(justify left)
+			)
+		)
+		(property "Footprint" "Diode_SMD:D_SMC"
+			(at 244.475 104.14 0)
+			(effects
+				(font
+					(size 1.27 1.27)
+				)
+				(hide yes)
+			)
+		)
+		(property "Datasheet" "http://www.jameco.com/Jameco/Products/ProdDS/1538777.pdf"
+			(at 248.92 104.14 0)
+			(effects
+				(font
+					(size 1.27 1.27)
+				)
+				(hide yes)
+			)
+		)
+		(property "Description" "60V 3A Schottky Barrier Rectifier Diode, SMC"
+			(at 248.92 104.14 0)
+			(effects
+				(font
+					(size 1.27 1.27)
+				)
+				(hide yes)
+			)
+		)
+		(pin "2"
+		)
+		(pin "1"
+		)
+		(instances
+			(project ""
+				(path "/2863b0a4-ce41-4b5d-85c6-a6fe5f63d9f6"
+					(reference "D3")
+					(unit 1)
+				)
+			)
+		)
+	)
+	(symbol
 		(lib_id "Device:C")
 		(at 59.69 162.56 90)
@@
 					(unit 1)
 				)
-			)
-		)
-	)
-	(symbol
-		(lib_id "Device:D_Schottky")
-		(at 248.92 104.14 270)
-		(unit 1)
-		(exclude_from_sim no)
-		(in_bom yes)
-		(on_board yes)
-		(dnp no)
-		(fields_autoplaced yes)
-		(property "Reference" "D4"
-			(at 251.46 102.5524 90)
-			(effects
-				(font
-					(size 1.27 1.27)
-				)
-				(justify left)
-			)
-		)
-		(property "Value" "D_Schottky"
-			(at 251.46 105.0924 90)
-			(effects
-				(font
-					(size 1.27 1.27)
-				)
-				(justify left)
-			)
-		)
-		(property "Footprint" ""
-			(at 248.92 104.14 0)
-			(effects
-				(font
-					(size 1.27 1.27)
-				)
-				(hide yes)
-			)
-		)
-		(property "Datasheet" "~"
-			(at 248.92 104.14 0)
-			(effects
-				(font
-					(size 1.27 1.27)
-				)
-				(hide yes)
-			)
-		)
-		(property "Description" "Schottky diode"
-			(at 248.92 104.14 0)
-			(effects
-				(font
-					(size 1.27 1.27)
-				)
-				(hide yes)
-			)
-		)
-		(pin "1"
-		)
-		(pin "2"
-		)
-		(instances
-			(project ""
-				(path "/2863b0a4-ce41-4b5d-85c6-a6fe5f63d9f6"
-					(reference "D4")
-					(unit 1)
-				)
