File: PCB/SunluS1Board/SunluS1Board.kicad_pcb (KiCad board)
At the start: 2 copper layers, 48.2 x 57 mm, 56 parts, among them J1 Conn_01x14, J2 aNTC, J3 hNTC, J4 Fan, J5 HT, J6 Power, J7 Conn_02x03_Odd_Even, Q1 SIA440DJ-T1-GE3, Q2 AO3400A, Q3 AO3400A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

Commit message: mostly finsish pcb, again
Parts:
- C17, C18, C19, C20, C21, C22, C5, D3, L1, R14, R15, R16, R17, R18, R19, U3: moved to F.Cu
- moved R18 14.0 mm to (105.7, 50.9)
- moved R14 12.3 mm to (104.8, 38.7), turned to 0 degrees
- moved R15 12.3 mm to (104.8, 37.1), turned to 180 degrees
- moved L1 12.1 mm to (92.7, 44.5), turned to 180 degrees
- moved C21 11.7 mm to (104.5, 53.9), turned to 0 degrees
- moved R17 11.7 mm to (104.5, 55.7), turned to 0 degrees
- moved C18 10.9 mm to (93.3, 47.9), turned to 0 degrees
- moved C19 10.9 mm to (93.3, 49.9), turned to 0 degrees
- moved R19 10.8 mm to (104.0, 41.5)
- moved C22 9.18 mm to (103.2, 43.9), turned to 180 degrees
- moved U3 8.57 mm to (102.9, 49.5)
- moved J7 7.69 mm to (89.9, 31.4)
- moved R16 7.10 mm to (102.2, 56.6)
- moved C5 5.53 mm to (101.4, 54.1), turned to 180 degrees
- moved C17 3.41 mm to (100.3, 51.8)
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Routing:
- net SWCLK: track 2.22 -> 26.8 mm, vias 1 -> 2
- net NRST: track 13.7 -> 37.1 mm
- net SWDIO: track 1.73 -> 23.2 mm, vias 1 -> 2
- net +3.3V: track 52.7 -> 49.3 mm, vias 5 -> 14
- net Net-(U3-COMP): track 8.13 -> 7.14 mm
- net GND: vias 26 -> 40
- added copper zone on F.Cu, net +24V
- added copper zone on F.Cu, net +3.3V
