File: PCB/SunluS1Board/SunluS1Board.kicad_pcb (KiCad board)
At the start: 2 copper layers, 48.2 x 57 mm, 56 parts, among them J1 Conn_01x14, J2 aNTC, J3 hNTC, J4 Fan, J5 HT, J6 Power, J7 Conn_02x03_Odd_Even, Q1 SIA440DJ-T1-GE3, Q2 AO3400A, Q3 AO3400A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

Commit message: finish V2
Parts:
- removed C16: 100uF, Capacitor_THT:CP_Radial_D6.3mm_P2.50mm
- added C6: 100uF, easyeda2kicad:CAP-SMD_BD6.3-L6.6-W6.6-FD, F.Cu at (95.3, 60.3)
- moved F1 0.80 mm to (98.5, 65.1)
Routing:
- net GND: track 55.3 -> 82.3 mm
- net +24V: track 48.3 -> 58.0 mm
- net B2: track 26.0 -> 28.2 mm
- net B1: track 26.1 -> 27.9 mm

Commit message: fix
Parts:
- C17, C5: value 0.1uF -> 100nF
Changed lines of the file:
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@@
 			)
 		)
-		(property "Value" "0.1uF"
+		(property "Value" "100nF"
 			(at 0 1.43 0)
 			(layer "F.Fab")
@@
 			)
 		)
-		(property "Value" "0.1uF"
+		(property "Value" "100nF"
 			(at 0 1.43 90)
 			(layer "F.Fab")

Commit message: fix
Parts:
- C6: value 100uF -> 47uF
Changed lines of the file:
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@@
 			)
 		)
-		(property "Value" "100uF"
+		(property "Value" "47uF"
 			(at 0 3.999999 30)
 			(layer "F.Fab")

Commit message: Fixes for V2
Parts:
- added D4: SS34, Diode_SMD:D_SMA, F.Cu at (79.6, 68.5)
- added D5: SS34, Diode_SMD:D_SMA, F.Cu at (87.8, 68.5)
- J4, J5, J6: footprint Connector_JST:JST_XH_S2B-XH-A-1_1x02_P2.50mm_Horizontal -> easyeda2kicad:CONN-TH_2P-P2.54_AXH-2AW-11
- moved J4 1.20 mm to (79.7, 72.0)
- moved J5 1.20 mm to (88.1, 72.0)
- moved J6 1.20 mm to (98.3, 72.0)
- moved C1 0.71 mm to (84.9, 65.8)
Routing:
- net GND: track 82.3 -> 90.7 mm, vias 40 -> 43
- net +24V: track 58.0 -> 65.8 mm
- net fCon: track 8.50 -> 12.3 mm
- net hCon: track 9.31 -> 10.5 mm
- net B2: track 28.2 -> 28.9 mm
